Commit message: [NextageOpen.urdf] Re-generated with robot_model 1.11.8 candidate.

File: nextage_description/urdf/NextageOpen.urdf (robot description, URDF)
Before this commit: robot NextageOpen, 16 links, 15 joints
Links:
- link WAIST: geometry collision mesh filename=package://nextage_description/urdf/meshes/WAIST_mesh.dae scale=1 1 1; visual mesh filename=package://nextage_description/urdf/meshes/WAIST_mesh.dae scale=1 1 1
Joints:
- joint CHEST_JOINT0: limit lower=-2.84489 upper=2.84489 effort=100 velocity=0.5 -> lower=-2.84489 upper=2.84489 effort=100 velocity=1.91986
- joint HEAD_JOINT0: limit lower=-1.22173 upper=1.22173 effort=100 velocity=0.5 -> lower=-1.22173 upper=1.22173 effort=100 velocity=2.61799
- joint HEAD_JOINT1: limit lower=-0.349066 upper=1.22173 effort=100 velocity=0.5 -> lower=-0.349066 upper=1.22173 effort=100 velocity=4.36332
- joint LARM_JOINT0: limit lower=-1.53589 upper=1.53589 effort=100 velocity=0.5 -> lower=-1.53589 upper=1.53589 effort=100 velocity=3.00197
- joint LARM_JOINT1: limit lower=-2.44346 upper=1.0472 effort=100 velocity=0.5 -> lower=-2.44346 upper=1.0472 effort=100 velocity=2.32129
- joint LARM_JOINT2: limit lower=-2.75762 upper=0 effort=100 velocity=0.5 -> lower=-2.75762 upper=0 effort=100 velocity=3.9968
- joint LARM_JOINT3: limit lower=-1.8326 upper=2.87979 effort=100 velocity=0.5 -> lower=-1.8326 upper=2.87979 effort=100 velocity=4.60767
- joint LARM_JOINT4: limit lower=-1.74533 upper=1.74533 effort=100 velocity=0.5 -> lower=-1.74533 upper=1.74533 effort=100 velocity=3.90954
- joint LARM_JOINT5: limit lower=-2.84489 upper=2.84489 effort=100 velocity=0.5 -> lower=-2.84489 upper=2.84489 effort=100 velocity=5.23599
- joint RARM_JOINT0: limit lower=-1.53589 upper=1.53589 effort=100 velocity=0.5 -> lower=-1.53589 upper=1.53589 effort=100 velocity=3.00197
- joint RARM_JOINT1: limit lower=-2.44346 upper=1.0472 effort=100 velocity=0.5 -> lower=-2.44346 upper=1.0472 effort=100 velocity=2.32129
- joint RARM_JOINT2: limit lower=-2.75762 upper=0 effort=100 velocity=0.5 -> lower=-2.75762 upper=0 effort=100 velocity=3.75246
- joint RARM_JOINT3: limit lower=-2.87979 upper=1.8326 effort=100 velocity=0.5 -> lower=-2.87979 upper=1.8326 effort=100 velocity=4.60767
- joint RARM_JOINT4: limit lower=-1.74533 upper=1.74533 effort=100 velocity=0.5 -> lower=-1.74533 upper=1.74533 effort=100 velocity=3.90954
- joint RARM_JOINT5: limit lower=-2.84489 upper=2.84489 effort=100 velocity=0.5 -> lower=-2.84489 upper=2.84489 effort=100 velocity=5.23599

Commit message: [NextageOpen.urdf] Re-apply the customizaion done in https://goo.gl/erZzwy

File: nextage_description/urdf/NextageOpen.urdf (robot description, URDF)
Before this commit: robot HiroNX, 16 links, 15 joints
Links:
- link WAIST: geometry collision mesh filename=package://nextage_description/urdf/meshes/WAIST_Link_mesh.d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 scale=1 1 1; visual mesh filename=package://nextage_description/urdf/meshes/WAIST_Link_mesh.d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 scale=1 1 1

Commit message: [gazebo] Add non-zero mass so that links are not ignored

File: nextage_description/urdf/NextageOpen.urdf (robot description, URDF)
Before this commit: robot NextageOpen, 16 links, 15 joints
Links:
- added link world
- link CHEST_JOINT0_Link: mass 0 -> 3.0
- link WAIST: mass 0 -> 30.0
Joints:
- added joint fixed: type fixed, parent world, child WAIST

File: nextage_gazebo/model/gazebo.xacro (robot description, xacro)
@@ -1,18 +1,6 @@
 <?xml version="1.0"?>
 <robot xmlns:xacro="http://www.ros.org/wiki/xacro">
-  <xacro:macro name="gazebo_base_link" params="name color">
-    <gazebo reference="${name}">
-      <!-- <material>Gazebo/${color}</material>  -->
-      <kp>100000.0</kp>
-      <kd>10.0</kd>
-      <mu1>1</mu1>
-      <mu2>1</mu2>
-      <fdir1>1 0 0</fdir1>
-      <minDepth>0.003</minDepth>
-      <maxVel>1.0</maxVel>
-    </gazebo>
-  </xacro:macro>
   <xacro:macro name="gazebo_nx_link" params="name color">
-    <gazebo reference="${name}">
+    <gazebo reference="gazebo_${name}">
       <material>Gazebo/${color}</material>
     </gazebo>

Commit message: set mass of base link to super hevey

File: nextage_description/urdf/NextageOpen.urdf (robot description, URDF)
Before this commit: robot NextageOpen, 16 links, 15 joints
Links:
- link WAIST: mass 30.0 -> 1000

Commit message: set ARM_JOINT1 max effor to 200, may be this is larget than real robot

File: nextage_description/urdf/NextageOpen.urdf (robot description, URDF)
Before this commit: robot NextageOpen, 16 links, 15 joints
Joints:
- joint LARM_JOINT1: limit lower=-2.44346 upper=1.0472 effort=100 velocity=0.5 -> lower=-2.44346 upper=1.0472 effort=200 velocity=0.5
- joint RARM_JOINT1: limit lower=-2.44346 upper=1.0472 effort=100 velocity=0.5 -> lower=-2.44346 upper=1.0472 effort=200 velocity=0.5

Commit message: set ARM_JOINT0 max effor to 150, may be this is larget than real robot

File: nextage_description/urdf/NextageOpen.urdf (robot description, URDF)
Before this commit: robot NextageOpen, 16 links, 15 joints
Joints:
- joint LARM_JOINT0: limit lower=-1.53589 upper=1.53589 effort=100 velocity=0.5 -> lower=-1.53589 upper=1.53589 effort=150 velocity=0.5
- joint RARM_JOINT0: limit lower=-1.53589 upper=1.53589 effort=100 velocity=0.5 -> lower=-1.53589 upper=1.53589 effort=150 velocity=0.5
