Commit message: fix package url in urdf files

File: nextage_calibration/models/checkerboard_horizontal.urdf (robot description, URDF)
Before this commit: robot checkeboard_horizontal, 2 links, 1 joints
Links:
- link checkerboard_base_link: geometry collision mesh filename=package://nextage_calibration/models/checkerboard_horizonta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; visual mesh filename=package://nextage_calibration/models/checkerboard_horizonta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

File: nextage_calibration/models/checkerboard_waist.urdf (robot description, URDF)
Before this commit: robot checkeboard_horizontal, 2 links, 1 joints
Links:
- link checkerboard_waist_base_link: geometry visual mesh filename=package://nextage_calibration/models/checkerboard_waist.dae
